File: ergogen/right/output/right/right.kicad_pcb (KiCad board)
At the start: 2 copper layers, 326.8 x 111 mm, 99 parts

Commit message: fixes
Routing:
- net VCC: track 24.8 -> 0.00 mm
- net P1: track 396.9 -> 372.7 mm
- net P0: track 385.1 -> 361.3 mm, vias 6 -> 5
- net P3: track 300.4 -> 306.2 mm, vias 5 -> 7
- net P2: track 331.3 -> 331.7 mm, vias 12 -> 14
